File: hardware/bus_simulator/bus_simulator.kicad_sch (KiCad schematic)
At the start: 47 parts, among them J1 I2C_LCD, J2 Encoder, SW1 SW_Push, U1 RaspberryPi_Pico, U2 74HC595, U3 74HC595, U4 74HC595

Commit message: Finished schematic
Parts:
- added D21, D22: LED, symbol Device:LED
- added R21, R22: 100, symbol Device:R
- added SW10, SW11, SW12, SW2, SW3, SW4, SW5, SW6, SW7, SW8, SW9: SW_Push, Button_Switch_SMD:SW_MEC_5GSH9, symbol Switch:SW_Push
Connections:
- net +3.3V: now also J2.5 (Pin_5), U1.36 (3V3)
- net GND: now also J2.1 (Pin_1), SW1.1, U1.13 (GND), U1.18 (GND), U1.23 (GND), U1.28 (GND), U1.3 (GND), U1.38 (GND), U1.8 (GND), D21.1 (K), D22.1 (K), SW10.1, SW11.1, SW12.1, SW2.1, SW3.1, SW4.1, SW5.1, SW6.1, SW7.1, SW8.1, SW9.1
- net at U1.1 (GPIO0): now also SW1.2; no longer J1.3 (Pin_3)
- net at U1.2 (GPIO1): now also SW2.2; no longer J1.4 (Pin_4)
- net at U4.4 (QE): now also R21.2
- net at U4.5 (QF): now also R22.2
- net at U1.10 (GPIO7): now also SW8.2
- net at U1.11 (GPIO8): now also SW9.2
- net at U1.12 (GPIO9): now also SW10.2
- net at U1.14 (GPIO10): now also SW11.2
- net at U1.15 (GPIO11): now also SW12.2
- net LCD_SDA: now reaches U1.16 (GPIO12)
- net LCD_SDA: now also J1.3 (Pin_3)
- net LCD_SCL: now reaches U1.17 (GPIO13)
- net LCD_SCL: now also J1.4 (Pin_4)
- net ENC_S1: now reaches U1.25 (GPIO19)
- net ENC_S1: now also J2.2 (Pin_2)
- net ENC_S2: now reaches U1.26 (GPIO20)
- net ENC_S2: now also J2.3 (Pin_3)
- net ENC_SW: now reaches U1.27 (GPIO21)
- net ENC_SW: now also J2.4 (Pin_4)
- net at U1.4 (GPIO2): now also SW3.2
- net at U1.5 (GPIO3): now also SW4.2
- net at U1.6 (GPIO4): now also SW5.2
- net at U1.7 (GPIO5): now also SW6.2
- net at U1.9 (GPIO6): now also SW7.2
- new net: D21.2 (A), R21.1
- new net: D22.2 (A), R22.1
Other:
- note added: "Bus data input"
- note added: "RAM address"
- note added: "RAM contnet"
- note added: "RAM data input"
- note added: "Ra/Rb/Rc"
- note added: "Rwy"
- moved on the sheet: D10, D11, D12, J1, J2, R10, R11, R12, SW1
